Commit message: release: reconstruct self-collision safety checkpoint

File: src/abb120_moveit_config1/config/gazebo_handarm.urdf (robot description, URDF)
Before this commit: robot handarm, 19 links, 18 joints
Links:
- link handbase_link: geometry collision mesh filename=package://handarmtest1/meshes/myhand/handbase_link_collisio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; visual mesh filename=package://handarmtest1/meshes/myhand/handbase_link.STL

File: src/abb120_moveit_config1/config/gazebo_handarm_velocity.urdf (robot description, URDF)
Before this commit: robot handarm, 19 links, 18 joints
Links:
- link handbase_link: geometry collision mesh filename=package://handarmtest1/meshes/myhand/handbase_link_collisio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; visual mesh filename=package://handarmtest1/meshes/myhand/handbase_link.STL

File: src/handarmtest1/urdf/arm.urdf (robot description, URDF)
Before this commit: robot handarm, 19 links, 18 joints
Links:
- link handbase_link: geometry collision mesh filename=package://handarmtest1/meshes/myhand/handbase_link_collisio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; visual mesh filename=package://handarmtest1/meshes/myhand/handbase_link.STL
Joints:
- joint joint_6: limit lower=-6.98132 upper=6.98132 effort=100 velocity=7.33038 -> lower=-6.981317 upper=6.981317 effort=100 velocity=7.33038

File: src/handarmtest1/xacro/hand.xacro (robot description, xacro)
@@ -35,11 +35,11 @@
       </material>
     </visual>
-    <collision>
-      <origin
-        xyz="0 0 0"
-        rpy="0 0 0" />
-      <geometry>
-        <mesh
-          filename="package://handarmtest1/meshes/myhand/handbase_link.STL" />
+    <!-- The former enclosing cylinder filled the finger-root cut-outs and
+         forced MoveIt to ignore real hand-base collision pairs.  This reduced
+         CAD mesh preserves the cut-outs while remaining practical at 60 Hz. -->
+    <collision>
+      <origin xyz="0 0 0" rpy="0 0 0" />
+      <geometry>
+        <mesh filename="package://handarmtest1/meshes/myhand/handbase_link_collision_8mm.STL" />
       </geometry>
     </collision>
@@ -82,11 +82,10 @@
     </visual>
     <collision>
-      <origin
-        xyz="0 0 0"
-        rpy="0 0 0" />
-      <geometry>
-        <mesh
-          filename="package://handarmtest1/meshes/myhand/f1link1.STL" />
-      </geometry>
+      <origin xyz="0 0 -0.0065" rpy="0 0 0" />
+      <geometry><cylinder radius="0.019" length="0.021" /></geometry>
+    </collision>
+    <collision>
+      <origin xyz="0.035 0.035 0.033" rpy="0 0 0.785398" />
+      <geometry><box size="0.083 0.042 0.066" /></geometry>
     </collision>
   </link>
@@ -106,6 +105,7 @@
       lower="0"
       upper="3.14"
-      effort="100"
-      velocity="4" />
+      effort="4.0"
+      velocity="0.8" />
+    <dynamics damping="0.05" friction="0.0" />
   </joint>
   <link
@@ -140,11 +140,14 @@
     </visual>
     <collision>
-      <origin
-        xyz="0 0 0"
-        rpy="0 0 0" />
-      <geometry>
-        <mesh
-          filename="package://handarmtest1/meshes/myhand/f1link2.STL" />
-      </geometry>
+      <origin xyz="0.01955 0.02385 0.0179" rpy="0 1.570796 0.8840" />
+      <geometry><cylinder radius="0.0179" length="0.06167" /></geometry>
+    </collision>
+    <collision>
+      <origin xyz="0 0 0.0179" rpy="0 0 0" />
+      <geometry><sphere radius="0.0179" /></geometry>
+    </collision>
+    <collision>
+      <origin xyz="0.0391 0.0477 0.0179" rpy="0 0 0" />
+      <geometry><sphere radius="0.0179" /></geometry>
     </collision>
   </link>
@@ -164,6 +167,7 @@
       lower="0"
       upper="1.3963"
-      effort="100"
-      velocity="4" />
+      effort="2.0"
+      velocity="0.8" />
+    <dynamics damping="0.04" friction="0.0" />
   </joint>
   <link
@@ -198,16 +202,19 @@
     </visual>
     <collision>
-      <origin
-        xyz="0 0 0"
-        rpy="0 0 0" />
-      <geometry>
-        <mesh
-          filename="package://handarmtest1/meshes/myhand/f1link3.STL" />
-      </geometry>
+      <origin xyz="0.014835 0.025415 0.012" rpy="0 1.570796 1.0425" />
+      <geometry><cylinder radius="0.0125" length="0.05886" /></geometry>
+    </collision>
+    <collision>
+      <origin xyz="0 0 0.012" rpy="0 0 0" />
+      <geometry><sphere radius="0.0125" /></geometry>
+    </collision>
+    <collision>
+      <origin xyz="0.02967 0.05083 0.012" rpy="0 0 0" />
+      <geometry><sphere radius="0.0125" /></geometry>
     </collision>
   </link>
   <joint
     name="f1j3"
-    type="continuous">
+    type="revolute">
     <origin
       xyz="0.044995 0.053623 0.007"
@@ -221,7 +228,8 @@
     <limit
       lower="0"
-      upper="0"
-      effort="100"
-      velocity="4" />
+      upper="1.3963"
+      effort="2.0"
+      velocity="0.8" />
+    <dynamics damping="0.01" friction="0.0" />
     <mimic
       joint="f1j2"
@@ -260,16 +268,15 @@
     </visual>
     <collision>
-      <origin
-        xyz="0 0 0"
-        rpy="0 0 0" />
-      <geometry>
-        <mesh
-          filename="package://handarmtest1/meshes/myhand/f3link1.STL" />
-      </geometry>
+      <origin xyz="0 0 0.0065" rpy="0 0 0" />
+      <geometry><cylinder radius="0.019" length="0.021" /></geometry>
+    </collision>
+    <collision>
+      <origin xyz="-0.035 0.035 -0.033" rpy="0 0 2.356194" />
+      <geometry><box size="0.083 0.042 0.066" /></geometry>
     </collision>
   </link>
   <joint
     name="f3j1"
-    type="continuous">
+    type="revolute">
     <origin
       xyz="0.029404 -0.02886 0.10643"
@@ -283,7 +290,8 @@
     <limit
       lower="0"
-      upper="0"
-      effort="100"
-      velocity="4" />
+      upper="3.14"
+      effort="4.0"
+      velocity="0.8" />
+    <dynamics damping="0.05" friction="0.0" />
     <mimic
       joint="f1j1"
@@ -322,11 +330,14 @@
     </visual>
     <collision>
-      <origin
-        xyz="0 0 0"
-        rpy="0 0 0" />
-      <geometry>
-        <mesh
-          filename="package://handarmtest1/meshes/myhand/f3link2.STL" />
-      </geometry>
+      <origin xyz="0.01955 0.02385 0.0179" rpy="0 1.570796 0.8840" />
+      <geometry><cylinder radius="0.0179" length="0.06167" /></geometry>
+    </collision>
+    <collision>
+      <origin xyz="0 0 0.0179" rpy="0 0 0" />
+      <geometry><sphere radius="0.0179" /></geometry>
+    </collision>
+    <collision>
+      <origin xyz="0.0391 0.0477 0.0179" rpy="0 0 0" />
+      <geometry><sphere radius="0.0179" /></geometry>
     </collision>
   </link>
@@ -346,6 +357,7 @@
       lower="0"
       upper="1.3963"
-      effort="100"
-      velocity="4" />
+      effort="2.0"
+      velocity="0.8" />
+    <dynamics damping="0.04" friction="0.0" />
   </joint>
   <link
@@ -380,16 +392,19 @@
     </visual>
     <collision>
-      <origin
-        xyz="0 0 0"
-        rpy="0 0 0" />
-      <geometry>
-        <mesh
-          filename="package://handarmtest1/meshes/myhand/f3link3.STL" />
-      </geometry>
+      <origin xyz="0.014835 0.025415 0.012" rpy="0 1.570796 1.0425" />
+      <geometry><cylinder radius="0.0125" length="0.05886" /></geometry>
+    </collision>
+    <collision>
+      <origin xyz="0 0 0.012" rpy="0 0 0" />
+      <geometry><sphere radius="0.0125" /></geometry>
+    </collision>
+    <collision>
+      <origin xyz="0.02967 0.05083 0.012" rpy="0 0 0" />
+      <geometry><sphere radius="0.0125" /></geometry>
     </collision>
   </link>
   <joint
     name="f3j3"
-    type="continuous">
+    type="revolute">
     <origin
       xyz="0.044995 0.053623 0.007"
@@ -403,7 +418,8 @@
     <limit
       lower="0"
-      upper="0"
-      effort="100"
-      velocity="4" />
+      upper="1.3963"
+      effort="2.0"
+      velocity="0.8" />
+    <dynamics damping="0.01" friction="0.0" />
     <mimic
       joint="f3j2"
@@ -442,11 +458,14 @@
     </visual>
     <collision>
-      <origin
-        xyz="0 0 0"
-        rpy="0 0 0" />
-      <geometry>
-        <mesh
-          filename="package://handarmtest1/meshes/myhand/f2link1.STL" />
-      </geometry>
+      <origin xyz="0.01955 0.02385 0.0179" rpy="0 1.570796 0.8840" />
+      <geometry><cylinder radius="0.0179" length="0.06167" /></geometry>
+    </collision>
+    <collision>
+      <origin xyz="0 0 0.0179" rpy="0 0 0" />
+      <geometry><sphere radius="0.0179" /></geometry>
+    </collision>
+    <collision>
+      <origin xyz="0.0391 0.0477 0.0179" rpy="0 0 0" />
+      <geometry><sphere radius="0.0179" /></geometry>
     </collision>
   </link>
@@ -466,6 +485,7 @@
       lower="0"
       upper="1.3963"
-      effort="100"
-      velocity="4" />
+      effort="2.0"
+      velocity="0.8" />
+    <dynamics damping="0.04" friction="0.0" />
   </joint>
   <link
@@ -500,16 +520,19 @@
     </visual>
     <collision>
-      <origin
-        xyz="0 0 0"
-        rpy="0 0 0" />
-      <geometry>
-        <mesh
-          filename="package://handarmtest1/meshes/myhand/f2link2.STL" />
-      </geometry>
+      <origin xyz="0.014835 0.025415 0.012" rpy="0 1.570796 1.0425" />
+      <geometry><cylinder radius="0.0125" length="0.05886" /></geometry>
+    </collision>
+    <collision>
+      <origin xyz="0 0 0.012" rpy="0 0 0" />
+      <geometry><sphere radius="0.0125" /></geometry>
+    </collision>
+    <collision>
+      <origin xyz="0.02967 0.05083 0.012" rpy="0 0 0" />
+      <geometry><sphere radius="0.0125" /></geometry>
     </collision>
   </link>
   <joint
     name="f2j2"
-    type="continuous">
+    type="revolute">
     <origin
       xyz="0.044995 0.053623 0.0058"
@@ -523,7 +546,8 @@
     <limit
       lower="0"
-      upper="0"
-      effort="100"
-      velocity="4" />
+      upper="1.3963"
+      effort="2.0"
+      velocity="0.8" />
+    <dynamics damping="0.01" friction="0.0" />
     <mimic
       joint="f2j1"
@@ -531,3 +555,15 @@
       offset="0" />
   </joint>
+  <!-- Physics-level backstop. MoveIt/SRDF remains the predictive command
+       gate; Gazebo contact must still prevent non-parent links from passing
+       through one another if a command-side defect ever escapes that gate. -->
+  <gazebo reference="handbase_link"><selfCollide>true</selfCollide></gazebo>
+  <gazebo reference="f1link1"><selfCollide>true</selfCollide></gazebo>
+  <gazebo reference="f1link2"><selfCollide>true</selfCollide></gazebo>
+  <gazebo reference="f1link3"><selfCollide>true</selfCollide></gazebo>
+  <gazebo reference="f2link1"><selfCollide>true</selfCollide></gazebo>
+  <gazebo reference="f2link2"><selfCollide>true</selfCollide></gazebo>
+  <gazebo reference="f3link1"><selfCollide>true</selfCollide></gazebo>
+  <gazebo reference="f3link2"><selfCollide>true</selfCollide></gazebo>
+  <gazebo reference="f3link3"><selfCollide>true</selfCollide></gazebo>
 </robot>

Commit message: fix: restore collision-safe arm control path

File: src/abb120_moveit_config1/config/gazebo_handarm.urdf (robot description, URDF)
Before this commit: robot handarm, 19 links, 18 joints
Links:
- link handbase_link: geometry collision mesh filename=package://handarmtest1/meshes/myhand/handbase_link_collisio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; visual mesh filename=package://handarmtest1/meshes/myhand/handbase_link.STL

File: src/handarmtest1/xacro/hand_g.xacro (robot description, xacro)
@@ -40,37 +40,45 @@
   <gazebo reference="handbase_link">
     <material>Gazebo/Black</material>
-    <turnGravityOff>true</turnGravityOff>
+    <turnGravityOff>false</turnGravityOff>
   </gazebo>
   <gazebo reference="f1link1">
     <material>Gazebo/Grey</material>
-    <turnGravityOff>true</turnGravityOff>
+    <turnGravityOff>false</turnGravityOff>
+    <mu1>1.5</mu1><mu2>1.5</mu2>
   </gazebo>
   <gazebo reference="f1link2">
     <material>Gazebo/Grey</material>
-    <turnGravityOff>true</turnGravityOff>
+    <turnGravityOff>false</turnGravityOff>
+    <mu1>1.5</mu1><mu2>1.5</mu2>
   </gazebo>
   <gazebo reference="f1link3">
     <material>Gazebo/Grey</material>
-    <turnGravityOff>true</turnGravityOff>
+    <turnGravityOff>false</turnGravityOff>
+    <mu1>1.5</mu1><mu2>1.5</mu2>
   </gazebo>
   <gazebo reference="f2link1">
     <material>Gazebo/Grey</material>
-    <turnGravityOff>true</turnGravityOff>
+    <turnGravityOff>false</turnGravityOff>
+    <mu1>1.5</mu1><mu2>1.5</mu2>
   </gazebo>
   <gazebo reference="f2link2">
     <material>Gazebo/Grey</material>
-    <turnGravityOff>true</turnGravityOff>
+    <turnGravityOff>false</turnGravityOff>
+    <mu1>1.5</mu1><mu2>1.5</mu2>
   </gazebo>
   <gazebo reference="f3link1">
     <material>Gazebo/Grey</material>
-    <turnGravityOff>true</turnGravityOff>
+    <turnGravityOff>false</turnGravityOff>
+    <mu1>1.5</mu1><mu2>1.5</mu2>
   </gazebo>
   <gazebo reference="f3link2">
     <material>Gazebo/Grey</material>
-    <turnGravityOff>true</turnGravityOff>
+    <turnGravityOff>false</turnGravityOff>
+    <mu1>1.5</mu1><mu2>1.5</mu2>
   </gazebo>
   <gazebo reference="f3link3">
     <material>Gazebo/Grey</material>
-    <turnGravityOff>true</turnGravityOff>
+    <turnGravityOff>false</turnGravityOff>
+    <mu1>1.5</mu1><mu2>1.5</mu2>
   </gazebo>
 </robot>

Commit message: Freeze whole-wrist teleoperation with four scene presets

File: src/abb120_moveit_config1/config/gazebo_handarm.urdf (robot description, URDF)
Before this commit: robot handarm, 19 links, 18 joints
Joints:
- joint link_6-tool0: origin xyz=0.17 0 0 rpy=0 1.5707963267948966 0 -> xyz=0.1658 0 0 rpy=0 1.5707963267948966 0

File: src/abb120_moveit_config1/config/gazebo_handarm_velocity.urdf (robot description, URDF)
Before this commit: robot handarm, 19 links, 18 joints
Joints:
- joint link_6-tool0: origin xyz=0.17 0 0 rpy=0 1.5707963267948966 0 -> xyz=0.1658 0 0 rpy=0 1.5707963267948966 0

File: src/handarmtest1/urdf/arm.urdf (robot description, URDF)
Before this commit: robot handarm, 19 links, 18 joints
Joints:
- joint link_6-tool0: origin xyz=0.17 0 0 rpy=0 1.5707963267948966 0 -> xyz=0.1658 0 0 rpy=0 1.5707963267948966 0

File: src/handarmtest1/xacro/arm_macro.xacro (robot description, xacro)
@@ -221,8 +221,8 @@
       <child link="${prefix}flange"/>
     </joint>
-    <!-- ROS-Industrial 'tool0' frame: all-zeros tool frame -->
+    <!-- Palm-surface control point: user-selected 165.8 mm axial offset. -->
     <link name="${prefix}tool0" />
     <joint name="${prefix}link_6-tool0" type="fixed">
-      <origin xyz="0.17 0 0" rpy="0 ${radians(90)} 0" />
+      <origin xyz="0.1658 0 0" rpy="0 ${radians(90)} 0" />
       <parent link="${prefix}flange" />
       <child link="${prefix}tool0" />
